File: PCB/HackPad.kicad_pcb (KiCad board)
At the start: 2 copper layers, 78 x 100 mm, 50 parts, among them J1 0.91 OLED Display, SW1 MX, SW10 MX, SW11 MX, SW12 MX, SW13 MX, SW14 MX, SW15 MX, SW16 MX, SW2 MX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

Commit message: Add files via upload
Parts:
- added REF**: MountingHole_3.2mm_M3, MountingHole:MountingHole_3.2mm_M3, F.Cu at (45.0, 34.0)
- added REF**: MountingHole_3.2mm_M3, MountingHole:MountingHole_3.2mm_M3, F.Cu at (80.0, 110.0)
- added REF**: MountingHole_3.2mm_M3, MountingHole:MountingHole_3.2mm_M3, F.Cu at (87.0, 45.2)
Routing:
- net GND: vias 50 -> 49

Commit message: Add files via upload
Parts:
- moved REF** 3.09 mm to (90.0, 46.0)
Routing:
- net VBUS: track 304.5 -> 463.0 mm, vias 0 -> 3
- net ROW4: track 82.3 -> 144.4 mm
- net ROW3: track 60.3 -> 120.5 mm
- net ROW2: track 38.4 -> 98.5 mm
- net GND: track 21.2 -> 34.0 mm
